File: notAnArduino.kicad_pcb (KiCad board)
At the start: 2 copper layers, 20 parts, among them J1 PORTC, J2 PORTD, J3 PORTB, J4 AVR_ISP, J5 DC_IN, SW1 SW_RST, U1 ATmega328P-AU, U2 LM1117-5.0, Y1 8MHz Crystal

Commit message: foo
Parts:
- moved SW1 45.4 mm to (179.3, 94.5)
- moved C3 41.1 mm to (161.8, 90.9), turned to 270 degrees
- moved U2 40.7 mm to (171.4, 85.9), turned to 0 degrees
- moved R3 38.6 mm to (174.2, 94.5), turned to 270 degrees
- moved D1 36.9 mm to (181.9, 89.0), turned to 270 degrees
- moved J5 36.1 mm to (148.3, 87.9), turned to 270 degrees
- moved R1 32.6 mm to (178.3, 89.1), turned to 90 degrees
- moved C6 28.8 mm to (161.8, 81.8), turned to 90 degrees
- moved D2 6.74 mm to (179.3, 83.3)
- moved R2 5.55 mm to (182.4, 83.8), turned to 90 degrees
- moved J2 3.70 mm to (163.6, 63.5)
- moved C2 1.14 mm to (173.7, 64.5), turned to 270 degrees
Routing:
- net +5V: track 68.2 -> 116.9 mm
- net Net-(J2-Pad7): track 0.00 -> 29.5 mm
- net Net-(J2-Pad8): track 0.00 -> 27.0 mm
- net Net-(J2-Pad6): track 0.00 -> 25.3 mm
- net Net-(J2-Pad1): track 0.00 -> 21.3 mm
- net Net-(J2-Pad3): track 0.00 -> 15.7 mm
- net Net-(J2-Pad2): track 0.00 -> 15.7 mm
- net Net-(J2-Pad5): track 0.00 -> 15.3 mm
- net Net-(J2-Pad4): track 0.00 -> 11.2 mm
- net /NRST: track 122.6 -> 117.5 mm
- net /LED1: track 15.5 -> 16.4 mm
- added copper zone on B.Cu, net GND

Commit message: re layed out?? hehe
Parts:
- moved R3 79.1 mm to (246.9, 63.2)
- moved SW1 78.4 mm to (251.2, 63.2)
- moved J5 63.6 mm to (206.8, 62.7), turned to 180 degrees
- moved Y1 56.9 mm to (228.6, 71.1)
- moved J4 56.6 mm to (244.1, 73.7), turned to 180 degrees
- moved J2 56.0 mm to (219.5, 66.8)
- moved U1 55.9 mm to (236.2, 64.0)
- moved C2 55.4 mm to (229.1, 64.2)
- moved C1 54.8 mm to (242.6, 65.0), turned to 90 degrees
- moved C4 54.5 mm to (224.8, 69.8), turned to 90 degrees
- moved J1 54.5 mm to (246.4, 54.1)
- moved R1 52.2 mm to (229.9, 81.1), turned to 270 degrees
- moved J3 52.0 mm to (240.5, 84.3)
- moved C6 50.5 mm to (211.8, 74.7), turned to 180 degrees
- moved C5 50.1 mm to (224.8, 73.0), turned to 270 degrees
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Routing:
- net /NRST: track 117.5 -> 53.5 mm
- net +5V: track 116.9 -> 70.0 mm
- net /SPI_SCK: track 36.8 -> 25.0 mm
- net /SPI_MOSI: track 30.8 -> 20.0 mm
- net Net-(J2-Pad8): track 27.0 -> 18.4 mm
- net /VIN: track 15.0 -> 22.9 mm
- net Net-(J2-Pad7): track 29.5 -> 22.4 mm
- net Net-(J2-Pad6): track 25.3 -> 19.9 mm
- net /LED1: track 16.4 -> 20.7 mm
- net Net-(J1-Pad1): track 19.0 -> 14.8 mm
- net Net-(J3-Pad2): track 10.3 -> 14.5 mm
- net Net-(J1-Pad6): track 13.9 -> 9.91 mm
- net /XTO: track 9.21 -> 13.1 mm
- net /SPI_CS: track 15.0 -> 18.5 mm
- net Net-(J1-Pad2): track 18.6 -> 15.3 mm
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